File: keypad-pcb.kicad_sch (KiCad schematic)
At the start: 32 parts, among them J1 AVR-ISP-6, K1 SW_Push, K2 SW_Push, K3 SW_Push, K4 SW_Push, K5 SW_Push, K6 SW_Push, SW0 RESET, U1 ATmega32U4-A, Y1 XTAL

Commit message: some routing
Parts:
- K1, K2, K3, K4, K5, K6: footprint marbastlib-mx:SW_MX_HS_1u -> MX_Alps_Hybrid:MX-1U-NoLED
Changed lines of the file:
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@@
       (effects (font (size 1.27 1.27)) hide)
     )
-    (property "Footprint" "marbastlib-mx:SW_MX_HS_1u" (at 40.64 45.72 0)
+    (property "Footprint" "MX_Alps_Hybrid:MX-1U-NoLED" (at 40.64 45.72 0)
       (effects (font (size 1.27 1.27)) hide)
     )
@@
       (effects (font (size 1.27 1.27)) hide)
     )
-    (property "Footprint" "marbastlib-mx:SW_MX_HS_1u" (at 58.42 26.67 0)
+    (property "Footprint" "MX_Alps_Hybrid:MX-1U-NoLED" (at 58.42 26.67 0)
       (effects (font (size 1.27 1.27)) hide)
     )
@@
       (effects (font (size 1.27 1.27)) hide)
     )
-    (property "Footprint" "marbastlib-mx:SW_MX_HS_1u" (at 40.64 26.67 0)
+    (property "Footprint" "MX_Alps_Hybrid:MX-1U-NoLED" (at 40.64 26.67 0)
       (effects (font (size 1.27 1.27)) hide)
     )
@@
       (effects (font (size 1.27 1.27)) hide)
     )
-    (property "Footprint" "marbastlib-mx:SW_MX_HS_1u" (at 58.42 45.72 0)
+    (property "Footprint" "MX_Alps_Hybrid:MX-1U-NoLED" (at 58.42 45.72 0)
       (effects (font (size 1.27 1.27)) hide)
     )
@@
       (effects (font (size 1.27 1.27)) hide)
     )
-    (property "Footprint" "marbastlib-mx:SW_MX_HS_1u" (at 76.2 45.72 0)
+    (property "Footprint" "MX_Alps_Hybrid:MX-1U-NoLED" (at 76.2 45.72 0)
       (effects (font (size 1.27 1.27)) hide)
     )
@@
       (effects (font (size 1.27 1.27)) hide)
     )
-    (property "Footprint" "marbastlib-mx:SW_MX_HS_1u" (at 76.2 26.67 0)
-      (effects (font (size 1.27 1.27)) hide)
-    )
+    (property "Footprint" "MX_Alps_Hybrid:MX-1U-NoLED" (at 76.2 26.67 0)
+      (effects (font (size 1.27 1.27)) hide)
+    )

Commit message: clock+more
Parts:
- K1, K2, K3, K4, K5, K6: footprint MX_Alps_Hybrid:MX-1U-NoLED -> marbastlib-mx:SW_MX_HS_1u
Changed lines of the file:
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@@
       (effects (font (size 1.27 1.27)) hide)
     )
-    (property "Footprint" "MX_Alps_Hybrid:MX-1U-NoLED" (at 40.64 45.72 0)
+    (property "Footprint" "marbastlib-mx:SW_MX_HS_1u" (at 40.64 45.72 0)
       (effects (font (size 1.27 1.27)) hide)
     )
@@
       (effects (font (size 1.27 1.27)) hide)
     )
-    (property "Footprint" "MX_Alps_Hybrid:MX-1U-NoLED" (at 58.42 26.67 0)
+    (property "Footprint" "marbastlib-mx:SW_MX_HS_1u" (at 58.42 26.67 0)
       (effects (font (size 1.27 1.27)) hide)
     )
@@
       (effects (font (size 1.27 1.27)) hide)
     )
-    (property "Footprint" "MX_Alps_Hybrid:MX-1U-NoLED" (at 40.64 26.67 0)
+    (property "Footprint" "marbastlib-mx:SW_MX_HS_1u" (at 40.64 26.67 0)
       (effects (font (size 1.27 1.27)) hide)
     )
@@
       (effects (font (size 1.27 1.27)) hide)
     )
-    (property "Footprint" "MX_Alps_Hybrid:MX-1U-NoLED" (at 58.42 45.72 0)
+    (property "Footprint" "marbastlib-mx:SW_MX_HS_1u" (at 58.42 45.72 0)
       (effects (font (size 1.27 1.27)) hide)
     )
@@
       (effects (font (size 1.27 1.27)) hide)
     )
-    (property "Footprint" "MX_Alps_Hybrid:MX-1U-NoLED" (at 76.2 45.72 0)
+    (property "Footprint" "marbastlib-mx:SW_MX_HS_1u" (at 76.2 45.72 0)
       (effects (font (size 1.27 1.27)) hide)
     )
@@
       (effects (font (size 1.27 1.27)) hide)
     )
-    (property "Footprint" "MX_Alps_Hybrid:MX-1U-NoLED" (at 76.2 26.67 0)
-      (effects (font (size 1.27 1.27)) hide)
-    )
+    (property "Footprint" "marbastlib-mx:SW_MX_HS_1u" (at 76.2 26.67 0)
+      (effects (font (size 1.27 1.27)) hide)
+    )
