File: keypad-pcb.kicad_pcb (KiCad board)
At the start: 2 copper layers, 32 parts, among them J1 AVR-ISP-6, K1 SW_Push, K2 SW_Push, K3 SW_Push, K4 SW_Push, K5 SW_Push, K6 SW_Push, SW0 RESET, U1 ATmega32U4-A, Y1 XTAL

Commit message: some routing
Parts:
- K1, K2, K3, K4, K5, K6: footprint marbastlib-mx:SW_MX_HS_1u -> MX_Alps_Hybrid:MX-1U-NoLED
- moved R4 2.96 mm to (154.3, 105.0)
- moved J1 1.93 mm to (165.6, 109.4)
- moved C4 1.93 mm to (125.6, 108.5)
- moved C5 1.93 mm to (125.6, 111.5)
- moved C1 1.93 mm to (153.0, 111.5)
- moved C2 1.93 mm to (147.2, 113.9)
- moved C3 1.93 mm to (142.9, 127.5)
- moved C6 1.93 mm to (155.0, 118.0)
- moved C7 1.93 mm to (155.0, 120.4)
- moved R1 1.93 mm to (130.4, 126.7)
- moved R2 1.93 mm to (136.0, 108.2)
- moved R3 1.93 mm to (133.6, 108.2)
- moved SW0 1.93 mm to (166.9, 118.8)
- moved U1 1.93 mm to (136.8, 118.0)
- moved Y1 1.93 mm to (148.7, 118.8)
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Routing:
- net D-: track 0.00 -> 46.9 mm
- net D+: track 0.00 -> 46.8 mm
- net XTAL2: track 0.00 -> 5.41 mm
- net Net-(U1-D+): track 0.00 -> 3.51 mm
- net Net-(U1-D-): track 0.00 -> 3.50 mm
- net GND: track 0.00 -> 2.90 mm

Commit message: clock+more
Parts:
- K1, K2, K3, K4, K5, K6: footprint MX_Alps_Hybrid:MX-1U-NoLED -> marbastlib-mx:SW_MX_HS_1u
- moved C1 13.0 mm to (158.8, 123.2)
- moved C7 5.75 mm to (150.6, 116.7)
- moved C6 4.51 mm to (150.6, 119.1), turned to 0 degrees
- moved J1 2.11 mm to (167.2, 110.9)
- moved SW0 2.11 mm to (165.9, 120.7)
- moved Y1 2.08 mm to (146.8, 117.9), turned to 90 degrees
- moved C2 1.50 mm to (147.8, 112.5), turned to -90 degrees
- moved D3 1.12 mm to (141.3, 101.6)
- moved D7 1.12 mm to (122.2, 82.5)
- moved D2 1.12 mm to (160.3, 82.5)
- moved D5 1.12 mm to (122.2, 101.6)
- moved D4 1.12 mm to (160.3, 101.6)
- moved D6 1.08 mm to (141.3, 82.5)
- moved USB1 0.55 mm to (134.7, 53.9)
- moved K1 0.27 mm to (164.2, 78.0)
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Routing:
- net ROW1: track 0.00 -> 49.3 mm, vias 0 -> 3
- net ROW0: track 0.00 -> 48.5 mm, vias 0 -> 3
- net COL2: track 0.00 -> 21.4 mm
- net COL1: track 0.00 -> 21.4 mm
- net COL0: track 0.00 -> 21.4 mm
- net GND: track 2.90 -> 21.1 mm
- net XTAL1: track 0.00 -> 8.77 mm
- net Net-(D7-A): track 0.00 -> 8.27 mm
- net Net-(D5-A): track 0.00 -> 8.27 mm
- net Net-(D4-A): track 0.00 -> 8.27 mm
- net Net-(D3-A): track 0.00 -> 8.27 mm
- net Net-(D2-A): track 0.00 -> 8.27 mm
- net Net-(D6-A): track 0.00 -> 8.24 mm
- net XTAL2: track 5.41 -> 8.56 mm
- net D-: track 46.9 -> 49.7 mm
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
Commit message: complete routing
Parts:
- moved C1 23.9 mm to (139.2, 109.5), turned to 0 degrees
- moved C4 23.1 mm to (140.7, 126.0), turned to 0 degrees
- moved R4 19.9 mm to (149.1, 124.2), turned to 0 degrees
- moved F1 12.7 mm to (130.3, 67.3), turned to 180 degrees
- moved C3 12.2 mm to (130.8, 126.0), turned to 180 degrees
- moved R1 7.30 mm to (137.4, 128.8), turned to 0 degrees
- moved SW0 6.02 mm to (161.0, 124.2)
- moved J1 4.97 mm to (162.6, 112.8)
- moved R8 3.53 mm to (140.5, 65.0)
- moved R7 3.43 mm to (129.0, 65.0)
- moved C5 3.16 mm to (127.5, 114.0), turned to -90 degrees
Connections:
- U1 pad 37: COL2 -> COL0
- U1 pad 41: COL0 -> COL2
Routing:
- net +5V: track 0.00 -> 152.8 mm, vias 0 -> 7
- net COL1: track 21.4 -> 165.1 mm
- net GND: track 21.1 -> 139.0 mm, vias 0 -> 3
- net COL0: track 21.4 -> 139.1 mm
- net COL2: track 21.4 -> 92.2 mm, vias 0 -> 2
- net ROW0: track 48.5 -> 114.2 mm, vias 3 -> 4
- net RESET: track 0.00 -> 49.2 mm
- net ROW1: track 49.3 -> 90.7 mm, vias 3 -> 4
- net SCK: track 0.00 -> 33.0 mm
- net MISO: track 0.00 -> 25.2 mm
- net MOSI: track 0.00 -> 24.3 mm, vias 0 -> 1
- net Net-(U1-~{HWB}/PE2): track 0.00 -> 8.09 mm, vias 0 -> 2
- net VCC: track 0.00 -> 7.99 mm
- net Net-(USB1-CC1): track 0.00 -> 6.18 mm, vias 0 -> 2
- net Net-(USB1-CC2): track 0.00 -> 5.17 mm
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
Commit message: edge cut
Routing:
- added copper zone on B.Cu, net GND
- added copper zone on F.Cu, net GND
Other:
- board outline added: 72.4 x 83.1 mm
Changed lines of the file:
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@@
         (effects (font (size 1 1) (thickness 0.15)) (justify mirror))
     )
-    (fp_text value "HRO-TYPE-C-31-M-12" (at 0 -1.15) (layer "Dwgs.User")
+    (fp_text value "HRO-TYPE-C-31-M-12" (at -14.828 6.504) (layer "Dwgs.User")
         (effects (font (size 1 1) (thickness 0.15)))
     )
@@
     )
   )
+  (gr_line (start 140.208 58.42) (end 140.208 55.118)
+    (stroke (width 0.1) (type default)) (layer "Edge.Cuts"))
+  (gr_line (start 140.208 55.118) (end 129.286 55.118)
+    (stroke (width 0.1) (type default)) (layer "Edge.Cuts"))
+  (gr_line (start 129.286 58.42) (end 108.966 58.42)
+    (stroke (width 0.1) (type default)) (layer "Edge.Cuts"))
+  (gr_line (start 181.356 138.176) (end 181.356 58.42)
+    (stroke (width 0.1) (type default)) (layer "Edge.Cuts"))
+  (gr_line (start 129.286 55.118) (end 129.286 58.42)
+    (stroke (width 0.1) (type default)) (layer "Edge.Cuts"))
+  (gr_line (start 108.966 58.42) (end 108.966 138.176)
+    (stroke (width 0.1) (type default)) (layer "Edge.Cuts"))
+  (gr_line (start 108.966 138.176) (end 181.356 138.176)
+    (stroke (width 0.1) (type default)) (layer "Edge.Cuts"))
+  (gr_line (start 181.356 58.42) (end 140.208 58.42)
+    (stroke (width 0.1) (type default)) (layer "Edge.Cuts"))
   (segment (start 152.146 114.554) (end 151.892 114.3) (width 0.381) (layer "F.Cu") (net 1))
   (segment (start 154.686 114.554) (end 152.146 114.554) (width 0.381) (layer "F.Cu") (net 1))
@@
   (segment (start 132.2175 73.36375) (end 129.38125 76.2) (width 0.25) (layer "B.Cu") (net 28))
   (segment (start 131.3825 72.9625) (end 128.778 70.358) (width 0.25) (layer "B.Cu") (net 28))
+  (zone (net 1) (net_name "GND") (layer "F.Cu") (hatch edge 0.5)
+    (priority 2)
+    (connect_pads (clearance 0.5))
+    (min_thickness 0.25) (filled_areas_thickness no)
+    (fill (thermal_gap 0.5) (thermal_bridge_width 0.5))
+    (polygon
+      (pts
+        (xy 140.716 118.872)
+        (xy 144.78 118.872)
+        (xy 144.78 115.824)
+        (xy 140.716 115.824)
+      )
+    )
+  )
+  (zone (net 1) (net_name "GND") (layers "F&B.Cu") (hatch edge 0.5)
+    (priority 1)
+    (connect_pads (clearance 0.5))
+    (min_thickness 0.25) (filled_areas_thickness no)
+    (fill (thermal_gap 0.5) (thermal_bridge_width 0.5))
+    (polygon
+      (pts
+        (xy 141.478 113.284)
+        (xy 141.478 122.682)
+        (xy 132.08 122.682)
+        (xy 132.08 113.284)
+      )
+    )
+  )
+  (zone (net 1) (net_name "GND") (layers "F&B.Cu") (hatch edge 0.5)
+    (connect_pads (clearance 0.5))
+    (min_thickness 0.25) (filled_areas_thickness no)
+    (fill (thermal_gap 0.5) (thermal_bridge_width 0.5))
+    (polygon
+      (pts
+        (xy 143.51 109.982)
+        (xy 143.51 122.428)
+        (xy 154.432 122.428)
+        (xy 154.432 109.982)
+      )
+    )
+  )
 )
